File: encoder.kicad_sch (KiCad schematic)
At the start: 2 parts, among them IC2 AS5047P-ATSM

Commit message: Add MCU stuff, cortex debug connector and docs
Other:
- note removed: "Available modes: - SPI - ABI/Z - PWM - UVW Route only SPI mode, left the other pins NC Connect TEST pin to GND according to datasheet"
- moved on the sheet: C2, IC2
Changed lines of the file:
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@@
 		(company "CERN BE-CEM-EPR")
 	)
-	(text "Available modes:\n- SPI\n- ABI/Z\n- PWM\n- UVW\n\nRoute only SPI mode, left the other pins NC\n\nConnect TEST pin to GND according to datasheet"
+	(text "Decoupling\nCapacitor"
 		(exclude_from_sim no)
-		(at 123.698 55.88 0)
+		(at 90.678 72.898 0)
 		(effects
 			(font
@@
 		)
 	)
-	(text "Decoupling\nCapacitor"
+	(text_box "Available modes:\n- SPI\n- ABI/Z\n- PWM\n- UVW\n\nRoute only SPI mode, left the other pins NC\n\nConnect TEST pin to GND according to datasheet"
 		(exclude_from_sim no)
-		(at 86.868 70.358 0)
+		(at 120.65 69.85 0)
+		(size 71.12 20.32)
+		(margins 0.9525 0.9525 0.9525 0.9525)
+		(stroke
+			(width 0)
+			(type dot)
+		)
+		(fill
+			(type none)
+		)
 		(effects
 			(font
 				(size 1.27 1.27)
 			)
-			(justify left)
+			(justify left top)
 		)
 	)
 	(junction
-		(at 78.74 64.77)
+		(at 82.55 67.31)
 		(diameter 0)
 		(color 0 0 0 0)
 	)
 	(no_connect
-		(at 72.39 72.39)
+		(at 76.2 74.93)
 	)
 	(no_connect
-		(at 41.91 69.85)
+		(at 45.72 72.39)
 	)
 	(no_connect
-		(at 72.39 67.31)
+		(at 76.2 69.85)
 	)
 	(no_connect
-		(at 72.39 57.15)
+		(at 76.2 59.69)
 	)
 	(no_connect
-		(at 72.39 69.85)
+		(at 76.2 72.39)
 	)
 	(no_connect
-		(at 41.91 72.39)
+		(at 45.72 74.93)
 	)
 	(wire
 		(pts
-			(xy 72.39 62.23) (xy 78.74 62.23)
+			(xy 76.2 64.77) (xy 82.55 64.77)
 		)
 		(stroke
@@
 	(wire
 		(pts
-			(xy 78.74 62.23) (xy 78.74 64.77)
+			(xy 82.55 64.77) (xy 82.55 67.31)
 		)
 		(stroke
@@
 	(wire
 		(pts
-			(xy 72.39 64.77) (xy 78.74 64.77)
+			(xy 76.2 67.31) (xy 82.55 67.31)
 		)
 		(stroke
@@
 	(wire
 		(pts
-			(xy 78.74 64.77) (xy 85.09 64.77)
+			(xy 82.55 67.31) (xy 88.9 67.31)
 		)
 		(stroke
@@
 	(wire
 		(pts
-			(xy 78.74 67.31) (xy 78.74 64.77)
+			(xy 82.55 69.85) (xy 82.55 67.31)
 		)
 		(stroke
@@
 	(wire
 		(pts
-			(xy 78.74 72.39) (xy 78.74 73.66)
+			(xy 82.55 74.93) (xy 82.55 76.2)
 		)
 		(stroke
@@
 	)
 	(image
-		(at 160.02 29.21)
+		(at 156.718 54.356)
 		(scale 0.515742)
 		(data "iVBORw0KGgoAAAANSUhEUgAABmkAAAKVCAYAAAAk+A8yAAAgAElEQVR4XuzdB5gkVb338UPOIBkE"
@@
 	(hierarchical_label "ENCODER_MISO"
 		(shape input)
-		(at 41.91 62.23 180)
+		(at 45.72 64.77 180)
 		(effects
 			(font
@@
 	(hierarchical_label "ENCODER_CSn"
 		(shape input)
-		(at 41.91 57.15 180)
+		(at 45.72 59.69 180)
 		(effects
 			(font
@@
 	(hierarchical_label "ENCODER_MOSI"
 		(shape input)
-		(at 41.91 64.77 180)
+		(at 45.72 67.31 180)
 		(effects
 			(font
@@
 	(hierarchical_label "ENCODER_3V3"
 		(shape input)
-		(at 85.09 64.77 0)
+		(at 88.9 67.31 0)
 		(effects
 			(font
@@
 	(hierarchical_label "ENCODER_SCLK"
 		(shape input)
-		(at 41.91 59.69 180)
+		(at 45.72 62.23 180)
 		(effects
 			(font
@@
 	(symbol
 		(lib_id "Device:C_Small")
-		(at 78.74 69.85 0)
+		(at 82.55 72.39 0)
 		(unit 1)
 		(exclude_from_sim no)
@@
 		(fields_autoplaced yes)
 		(property "Reference" "C2"
-			(at 81.28 68.5862 0)
+			(at 85.09 71.1262 0)
 			(effects
 				(font
@@
 		)
 		(property "Value" "0.1u"
-			(at 81.28 71.1262 0)
+			(at 85.09 73.6662 0)
 			(effects
 				(font
@@
 		)
 		(property "Footprint" ""
-			(at 78.74 69.85 0)
+			(at 82.55 72.39 0)
 			(effects
 				(font
@@
 		)
 		(property "Datasheet" "~"
-			(at 78.74 69.85 0)
+			(at 82.55 72.39 0)
 			(effects
 				(font
@@
 		)
 		(property "Description" "Unpolarized capacitor, small symbol"
-			(at 78.74 69.85 0)
+			(at 82.55 72.39 0)
 			(effects
 				(font
@@
 	(symbol
 		(lib_id "power:GND")
-		(at 72.39 59.69 90)
+		(at 76.2 62.23 90)
 		(unit 1)
 		(exclude_from_sim no)
@@
 		(fields_autoplaced yes)
 		(property "Reference" "#PWR023"
-			(at 78.74 59.69 0)
+			(at 82.55 62.23 0)
 			(effects
 				(font
@@
 		)
 		(property "Value" "GND"
-			(at 76.2 59.6899 90)
+			(at 80.01 62.2299 90)
 			(effects
 				(font
@@
 		)
 		(property "Footprint" ""
-			(at 72.39 59.69 0)
+			(at 76.2 62.23 0)
 			(effects
 				(font
@@
 		)
 		(property "Datasheet" ""
-			(at 72.39 59.69 0)
+			(at 76.2 62.23 0)
 			(effects
 				(font
@@
 		)
 		(property "Description" "Power symbol creates a global label with name \"GND\" , ground"
-			(at 72.39 59.69 0)
+			(at 76.2 62.23 0)
 			(effects
 				(font
@@
 	(symbol
 		(lib_id "bldc-driver-pcb:AS5047P-ATSM")
-		(at 57.15 64.77 0)
+		(at 60.96 67.31 0)
 		(unit 1)
 		(exclude_from_sim no)
@@
 		(fields_autoplaced yes)
 		(property "Reference" "IC2"
-			(at 57.15 49.53 0)
+			(at 60.96 52.07 0)
 			(effects
 				(font
@@
 		)
 		(property "Value" "AS5047P-ATSM"
-			(at 57.15 52.07 0)
+			(at 60.96 54.61 0)
 			(effects
 				(font
@@
 		)
 		(property "Footprint" "bldc-driver-pcb:AS5047P"
-			(at 83.82 159.69 0)
+			(at 87.63 162.23 0)
 			(effects
 				(font
@@
 		)
 		(property "Datasheet" "https://datasheet.datasheetarchive.com/originals/distributors/DKDS-7/120640.pdf"
-			(at 83.82 259.69 0)
+			(at 87.63 262.23 0)
 			(effects
 				(font
@@
 		)
 		(property "Description" "Board Mount Hall Effect / Magnetic Sensors 14 bit core res Up to 28krpm"
-			(at 57.15 64.77 0)
+			(at 60.96 67.31 0)
 			(effects
 				(font
@@
 		)
 		(property "Height" "1.2"
-			(at 83.82 459.69 0)
+			(at 87.63 462.23 0)
 			(effects
 				(font
@@
 		)
 		(property "Mouser Part Number" "985-AS5047P-ATSM"
-			(at 83.82 559.69 0)
+			(at 87.63 562.23 0)
 			(effects
 				(font
@@
 		)
 		(property "Mouser Price/Stock" "https://www.mouser.co.uk/ProductDetail/ams-OSRAM/AS5047P-ATSM?qs=cGEy3R83DS8fzNOVLHtOgg%3D%3D"
-			(at 83.82 659.69 0)
+			(at 87.63 662.23 0)
 			(effects
 				(font
@@
 		)
 		(property "Manufacturer_Name" "ams OSRAM"
-			(at 83.82 759.69 0)
+			(at 87.63 762.23 0)
 			(effects
 				(font
@@
 		)
 		(property "Manufacturer_Part_Number" "AS5047P-ATSM"
-			(at 83.82 859.69 0)
+			(at 87.63 862.23 0)
 			(effects
 				(font
@@
 	(symbol
 		(lib_id "power:GND")
-		(at 41.91 67.31 270)
+		(at 45.72 69.85 270)
 		(unit 1)
 		(exclude_from_sim no)
@@
 		(fields_autoplaced yes)
 		(property "Reference" "#PWR022"
-			(at 35.56 67.31 0)
+			(at 39.37 69.85 0)
 			(effects
 				(font
@@
 		)
 		(property "Value" "GND"
-			(at 38.1 67.3099 90)
+			(at 41.91 69.8499 90)
 			(effects
 				(font
@@
 		)
 		(property "Footprint" ""
-			(at 41.91 67.31 0)
+			(at 45.72 69.85 0)
 			(effects
 				(font
@@
 		)
 		(property "Datasheet" ""
-			(at 41.91 67.31 0)
+			(at 45.72 69.85 0)
 			(effects
 				(font
@@
 		)
 		(property "Description" "Power symbol creates a global label with name \"GND\" , ground"
-			(at 41.91 67.31 0)
+			(at 45.72 69.85 0)
 			(effects
 				(font
@@
 	(symbol
 		(lib_id "power:GND")
-		(at 78.74 73.66 0)
+		(at 82.55 76.2 0)
 		(unit 1)
 		(exclude_from_sim no)
@@
 		(fields_autoplaced yes)
 		(property "Reference" "#PWR024"
-			(at 78.74 80.01 0)
+			(at 82.55 82.55 0)
 			(effects
 				(font
@@
 		)
 		(property "Value" "GND"
-			(at 78.74 78.74 0)
+			(at 82.55 81.28 0)
 			(effects
 				(font
@@
 		)
 		(property "Footprint" ""
-			(at 78.74 73.66 0)
+			(at 82.55 76.2 0)
 			(effects
 				(font
@@
 		)
 		(property "Datasheet" ""
-			(at 78.74 73.66 0)
+			(at 82.55 76.2 0)
 			(effects
 				(font
@@
 		)
 		(property "Description" "Power symbol creates a global label with name \"GND\" , ground"
-			(at 78.74 73.66 0)
-			(effects
-				(font
+			(at 82.55 76.2 0)
+			(effects
+				(font

Commit message: Initial routing
Parts:
- C2: footprint (none) -> Capacitor_SMD:C_0603_1608Metric
Changed lines of the file:
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@@
 			)
 		)
-		(property "Footprint" ""
+		(property "Footprint" "Capacitor_SMD:C_0603_1608Metric"
 			(at 82.55 72.39 0)
 			(effects
